Commit message: Add updates for gripper

File: xarm_description/urdf/xarm2.urdf (robot description, URDF)
Before this commit: robot xarm, 8 links, 7 joints
Links:
- added link xarm_1_joint
Joints:
- removed joint xarm_1_joint
- removed joint xarm_gripper_tip_joint
- added joint gripper_link_joint: type revolute, parent xarm_2_link, child xarm_1_link, origin xyz=0 0 0 rpy=0 0 0, axis 0 1 0, limit lower=-3.14 upper=3.14 effort=6 velocity=1

File: xarm_description/urdf/xarm2.urdf.xacro (robot description, xacro)
@@ -1,4 +1,4 @@
 <?xml version="1.0" ?>
-<robot name="xarm">
+<robot name="xarm" xmlns:xacro="http://ros.org/wiki/xacro">
     <material name="DarkGrey">
         <color rgba="0.3 0.3 0.3 1.0" />
@@ -162,6 +162,6 @@
         </inertial>
     </link>
-    <link name="xarm_gripper_tip" />
-    <!--link name="xarm_gripper_tip">
+    <!--link name="xarm_gripper_tip" /-->
+    <link name="xarm_gripper_tip">
         <visual>
             <origin rpy="0 0 0" xyz="0.0 0.0 0.0" />
@@ -181,5 +181,5 @@
             <inertia ixx="0.03" iyy="0.03" izz="0.03" ixy="0.0" ixz="0.0" iyz="0.0" />
         </inertial>
-    </link-->
+    </link>
     <joint name="xarm_6_joint" type="revolute">
         <origin rpy="0 0 0" xyz="0 0.0 0.03603" />
@@ -227,5 +227,16 @@
         <child link="xarm_2_link" />
     </joint>
-    <joint name="xarm_1_joint" type="revolute">
+    <!-- gripper_link -->
+    <!--link name="xarm_1_link"/-->
+    <!--joint name="xarm_1_joint" type="revolute">
+        <origin xyz="0 0 0" rpy="0 0 0"/>
+        <parent link="xarm_2_link"/>
+        <child link="xarm_1_link"/>
+        <limit effort="6" velocity="1" lower="-3.14" upper="3.14"/>
+        <axis xyz="0 1 0"/>
+    </joint-->
+    <!-- gripper -->
+    <!--xacro:include filename="$(find xarm_description)/urdf/xarm_gripper.xacro"/-->
+    <!--joint name="xarm_1_joint" type="revolute">
         <origin rpy="0 0 0" xyz="0 0 0.007548" />
         <axis xyz="0 0 1" />
@@ -238,5 +249,5 @@
       <child link = "xarm_gripper_tip" />
       <origin xyz="0.0 0.0 0.104639" rpy="0.0 0.0 0.0" />
-    </joint>
+    </joint-->
     <transmission name="trans_xarm_6_joint">
         <type>transmission_interface/SimpleTransmission</type>

File: xarm_description/urdf/xarm4.urdf.xacro (robot description, xacro)
@@ -1,4 +1,4 @@
 <?xml version="1.0" ?>
-<robot name="xarm">
+<robot name="xarm" xmlns:xacro="http://ros.org/wiki/xacro">
     <material name="DarkGrey">
         <color rgba="0.3 0.3 0.3 1.0" />
@@ -147,20 +147,20 @@
             <origin rpy="0 0 0" xyz="0.0 0.0 0.0" />
             <geometry>
-                <mesh filename="package://xarm_description/meshes/stls/gripper.stl" scale="1.0 1.0 1.0" />
-            </geometry>
-            <material name="DarkGrey" />
-        </visual>
-        <collision>
-            <origin rpy="0 0 0" xyz="0.0 0.0 0.0" />
-            <geometry>
-                <mesh filename="package://xarm_description/meshes/stls/gripper.stl" scale="1.0 1.0 1.0" />
-            </geometry>
-        </collision>
-        <inertial>
-            <mass value="0.1" />
-            <inertia ixx="0.03" iyy="0.03" izz="0.03" ixy="0.0" ixz="0.0" iyz="0.0" />
-        </inertial>
-    </link>
-    <link name="xarm_gripper_tip" />
+                <mesh filename="package://xarm_description/meshes/stls/ID1_servo.stl" scale=".001 .001 .001" />
+            </geometry>
+            <material name="DarkGrey" />
+        </visual>
+        <collision>
+            <origin rpy="0 0 0" xyz="0.0 0.0 0.0" />
+            <geometry>
+                <mesh filename="package://xarm_description/meshes/stls/ID1_servo.stl" scale=".001 .001 .001" />
+            </geometry>
+        </collision>
+        <inertial>
+            <mass value="0.1" />
+            <inertia ixx="0.03" iyy="0.03" izz="0.03" ixy="0.0" ixz="0.0" iyz="0.0" />
+        </inertial>
+    </link>
+    <!--link name="xarm_gripper_tip" /-->
     <!--link name="xarm_gripper_tip">
         <visual>
@@ -182,4 +182,6 @@
         </inertial>
     </link-->
+    <!-- gripper -->
+    <xacro:include filename="$(find xarm_description)/urdf/xarm_gripper.xacro"/>
     <joint name="xarm_6_joint" type="revolute">
         <origin rpy="0 0 0" xyz="0 0.0 0.03603" />
@@ -234,9 +236,10 @@
         <child link="xarm_1_link" />
     </joint>
-    <joint name="xarm_gripper_tip_joint" type="fixed">
+    <!--joint name="xarm_gripper_tip_joint" type="prismatic">
       <parent link="xarm_2_link" />
       <child link = "xarm_gripper_tip" />
+      <limit effort="30" velocity="0.5" lower="0.002" upper="0.042"/>
       <origin xyz="0.0 0.0 0.104639" rpy="0.0 0.0 0.0" />
-    </joint>
+    </joint-->
     <transmission name="trans_xarm_6_joint">
         <type>transmission_interface/SimpleTransmission</type>

File: xarm_description/urdf/xarm_world.urdf.xacro (robot description, xacro)
@@ -1,4 +1,4 @@
 <robot xmlns:xacro="http://ros.org/wiki/xacro" name="xarm">
-    <xacro:include filename="$(find xarm_description)/urdf/xarm.urdf"/>
+    <xacro:include filename="$(find xarm_description)/urdf/xarm4.urdf.xacro"/>
     <link name="world"/>
     <xacro:arg name="initial_z" default="0.0"/>
