Commit message: Add limits to mimic joints

File: xarm_description/urdf/xarm_gripper.xacro (robot description, xacro)
@@ -45,5 +45,5 @@
     <origin xyz="0 0 0.070" rpy="0 0 0"/>
     <axis xyz="1 0 0"/>
-    <limit effort="30" velocity="0.5" />
+    <limit effort="30" velocity="0.5" lower="0" upper="1" />
     <parent link="xarm_1_link"/>
     <child link="xarm_gripper_tip1"/>
@@ -58,5 +58,5 @@
     <origin xyz="0 0 0.070" rpy="0 0 0"/>
     <axis xyz="1 0 0"/>
-    <limit effort="30" velocity="0.5" />
+    <limit effort="30" velocity="0.5" lower="-1" upper="0" />
     <parent link="xarm_1_link"/>
     <child link="xarm_gripper_tip2"/>
