Commit message: Overwrite xarm config with fresh run

File: xarm_moveit_config/config/gazebo_xarm.urdf (robot description, URDF)
Before this commit: robot xarm, 7 links, 6 joints
Links:
- added link dummy_gripper_link
- added link xarm_gripper_tip1, mass 0.01; collision mesh filename=package://xarm_description/meshes/stls/right_finger-90.stl scale=.001 .001 .001; visual mesh filename=package://xarm_description/meshes/stls/right_finger-90.stl scale=.001 .001 .001
- added link xarm_gripper_tip2, mass 0.01; collision mesh filename=package://xarm_description/meshes/stls/right_finger-90.stl scale=.001 .001 .001; visual mesh filename=package://xarm_description/meshes/stls/right_finger-90.stl scale=.001 .001 .001
- link xarm_base_link: mass None -> 0.1
Joints:
- added joint xarm_1_joint: type prismatic, parent xarm_1_link, child dummy_gripper_link, origin xyz=0 0 0.070 rpy=0 0 0, axis 1 0 0, limit lower=0 upper=1 effort=30 velocity=0.5
- added joint xarm_tip1_joint: type prismatic, parent xarm_1_link, child xarm_gripper_tip1, origin xyz=0 0 0.070 rpy=0 0 0, axis 1 0 0, limit lower=0 upper=1 effort=30 velocity=0.5, mimic joint=xarm_1_joint multiplier=0.028 offset=0
- added joint xarm_tip2_joint: type prismatic, parent xarm_1_link, child xarm_gripper_tip2, origin xyz=0 0 0.070 rpy=0 0 0, axis 1 0 0, limit lower=-1 upper=0 effort=30 velocity=0.5, mimic joint=xarm_1_joint multiplier=-0.028 offset=0
